Commit message: 1. Set up rover_description package and launch files.  2. Created basic shape for rover.urdf/wheel.xacro

File: src/rover_description/urdf/rover.urdf (robot description, URDF)
Before this commit: robot myfirst, 1 links, 0 joints
Links:
- added link world
- link base_link: geometry visual box size=${length} ${width} ${height}
Joints:
- added joint world_joint: type fixed, parent world, child base_link, origin xyz=0 0 0 rpy=0 0 0
